File: LaserCutter.brd (EAGLE design)
At the start: 108.3 x 80.6 mm, 126 parts, among them IC1 ATMEGA8U2, IC10 LM393D, IC11 74AHC1G02DBV, IC12 74AHC1G02DBV, IC13 74AHC1G08DBV, IC14 MAX6675, IC2 BEE module, IC3 MC34063, IC4 74AHC1G02DBV, IC5 74AHC1G08DBV, IC6 ATMEGA2560-16AU, IC7 CD4050D, IC8 LD1117S33, IC9 OPA340N, J1 X Stepper, J10 Laser HV PSU, J11 24V in, J12 Interface, J13 I2C, J14 ISP, J15 SDMMC18650, J16 UART3, J17 X Home, J18 Z Home, J19 Y Home, J2 Reset En, J20 Interlocks, J21 Spare, J22 Omega PCC-SMP-V-K, J4 USB, J5 Y Stepper, J6 Ground, J7 ISP, J8 Z Stepper, J9 Stepper disable, Q1 16 MHz, Q2 16MHz

Commit message: foo
Parts:
- removed J22: Omega PCC-SMP-V-K, Thermocouple:TC_JACK
- added J3: USB, freetronics-master-v1:USB-MINIB-FT
- J10: value Laser HV PSU -> 24V in; device con-phoenix-254:4POL254 -> con-wago-508:W237-132
- J11: value 24V in -> Interface; device con-wago-508:W237-132 -> con-phoenix-254:8POL254
- J12: value Interface -> I2C; device con-phoenix-254:8POL254 -> freetronics-master-v1:1X02
- J13: value I2C -> SDMMC18650; device pinhead:1X02 -> adafruit:SDCARD
- J14: device SparkFun:2X3-NS -> freetronics-master-v1:2X03
- J15: value SDMMC18650 -> UART3; device adafruit:SDCARD -> freetronics-master-v1:1X02
- J16: value UART3 -> X Home; device pinhead:1X02 -> con-phoenix-254:3POL254
- J17: value X Home -> Z Home; device con-phoenix-254:3POL254 -> con-phoenix-254:5POL254
- J18: value Z Home -> Y Home; device con-phoenix-254:5POL254 -> con-phoenix-254:3POL254
- J19: value Y Home -> Interlocks; device con-phoenix-254:3POL254 -> con-phoenix-254:2POL254
- J20: value Interlocks -> Spare
- J21: value Spare -> Omega PCC-SMP-V-K; device con-phoenix-254:2POL254 -> freetronics-luke:PCC-SMP-V
- J4: value USB -> Y Stepper; device freetronics-master-v1:USB-MINIB-FT -> con-phoenix-254:6POL254
- J5: value Y Stepper -> Ground; device con-phoenix-254:6POL254 -> jumper:SJ
- J6: value Ground -> ISP; device jumper:SJ -> freetronics-master-v1:2X03
- J7: value ISP -> Z Stepper; device SparkFun:2X3-NS -> con-phoenix-254:6POL254
- J8: value Z Stepper -> Stepper disable; device con-phoenix-254:6POL254 -> wirepad:1,6/0,8
- J9: value Stepper disable -> Laser HV PSU; device wirepad:1,6/0,8 -> con-phoenix-254:4POL254
- moved J10 104.8 mm to (98.4, 73.7), turned to 0 degrees
- moved J21 91.9 mm to (91.8, 40.6), turned to 90 degrees
- moved J5 79.7 mm to (14.3, 11.4), flipped to the bottom, turned to 0 degrees
- moved J9 79.0 mm to (6.03, 24.1), turned to 270 degrees
- moved J4 77.6 mm to (66.4, 71.8), turned to 180 degrees
- moved J15 75.6 mm to (13.0, 60.6), turned to 0 degrees
- moved J7 72.5 mm to (84.1, 71.8), turned to 180 degrees
- moved J19 60.0 mm to (6.03, 14.6), turned to 270 degrees
- moved J13 58.8 mm to (75.9, 18.7), turned to 90 degrees
- moved J12 58.1 mm to (39.4, 63.5), turned to 180 degrees
- moved J16 22.9 mm to (34.6, 71.8), turned to 180 degrees
- moved J17 22.9 mm to (11.7, 71.8)
- moved J6 19.8 mm to (28.9, 24.8), flipped to the top, turned to 270 degrees
- moved J11 17.2 mm to (97.1, 56.5), turned to 90 degrees
- moved J8 13.3 mm to (75.6, 61.6), turned to 0 degrees
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- renumbered $0000002 to $1
Connections:
- net !8U2_RESET: now also J6.5; no longer J7.5
- net !DOOR: now also J19.1, J9.2; no longer J10.2, J20.1
- net !LASER_ENABLE: now also J9.1; no longer J10.1
- net !SD_CD: now also J13.CD; no longer J15.CD
- net !UI_CS: now also J11.8; no longer J12.8
- net +24V: now also J10.1, J16.1, J4.6, J7.6; no longer J11.1, J19.1, J5.6, J8.6
- net +3V3: now also J13.4; no longer J15.4
- net +5V: now also J11.1, J17.2, J4.3, J6.2, J7.3; no longer J12.1, J18.2, J5.3, J7.2, J8.3
- net 8U2_MISO: now also J6.1; no longer J7.1
- net 8U2_MOSI: now also J6.4; no longer J7.4
- net 8U2_SCK: now also J6.3; no longer J7.3
- net GND: now also J10.2, J13.3, J13.6, J13.COM, J13.MT1, J16.3, J17.5, J18.3, J20.2, J21.P$1, J21.P$2, J21.T-, J4.5, J5.2, J6.6, J7.5, J9.3; no longer J10.3, J12.2, J15.3, J15.6, J15.COM, J15.MT1, J17.3, J18.5, J19.3, J21.2, J22.P$1, J22.P$2, J22.T-, J5.5, J6.2, J7.6, J8.5
- net J81: now also J4.4, J7.4, J8.1; no longer J5.4, J8.4, J9.1
- net LASER_MODULATION: now also J9.4; no longer J10.4
- net MISO: now also J11.5, J13.7; no longer J12.5, J15.7
- net MOSI: now also J11.6; no longer J12.6
- net N$1: now also J13.2; no longer J15.2
- net N$101: now also J3.D-; no longer J4.D-
- net N$12: now also J19.2, J20.1; no longer J20.2, J21.1
- net N$120: now also J3.SH1, J3.SH2, J3.SH3, J3.SH4; no longer J4.SH1, J4.SH2, J4.SH3, J4.SH4
- net N$19: now also J13.1; no longer J15.1
- net N$25: now also J21.T+; no longer J22.T+
- net N$35: now also J17.3; no longer J18.3
- net N$6: now also J3.GND, J5.1; no longer J4.GND, J6.1
- net N$9: now also J13.5; no longer J15.5
- net N$97: now also J3.VBUS; no longer J4.VBUS
- net N$98: now also J3.D+; no longer J4.D+
- net RXD3: now also J15.1; no longer J16.1
- net SCK: now also J11.7; no longer J12.7
- net SCL: now also J12.2; no longer J13.2
- net SDA: now also J12.1; no longer J13.1
- net TXD3: now also J15.2; no longer J16.2
- net UI_RXD: now also J11.3; no longer J12.3
- net UI_TXD: now also J11.4; no longer J12.4
- net X_HOME: now also J16.2; no longer J17.2
- net Y_DIR: now also J4.2; no longer J5.2
- net Y_HOME: now also J18.2; no longer J19.2
- net Y_STEP: now also J4.1; no longer J5.1
- net Z_DIR: now also J7.2; no longer J8.2
- net Z_HOME: now also J17.4; no longer J18.4
- net Z_STEP: now also J7.1; no longer J8.1
Routing:
- net N$120: track 34.0 -> 32.7 mm
- net GND: track 40.4 -> 39.2 mm
- net +24V: track 226.0 -> 226.7 mm
- net N$8: track 10.9 -> 11.6 mm
- net N$21: track 11.6 -> 12.1 mm

Commit message: a few tweaks
Parts:
- moved C14 0.95 mm to (72.4, 41.9)
- moved J10 0.63 mm to (98.4, 73.0)
Connections:
- new net DAT1: J13.8
- new net DAT2: J13.9
- new net WP: J13.WP
Routing:
- net DAT1: track 0.00 -> 4.32 mm, vias 0 -> 4
- net N$9: track 27.5 -> 31.1 mm, vias 2 -> 6
- net N$120: track 32.7 -> 36.1 mm, vias 0 -> 6
- net DAT2: track 0.00 -> 3.13 mm, vias 0 -> 4
- net N$1: track 30.8 -> 33.8 mm, vias 0 -> 4
- net +3V3: track 79.8 -> 82.8 mm, vias 3 -> 7
- net N$19: track 60.8 -> 62.8 mm, vias 2 -> 6
- net WP: track 0.00 -> 1.97 mm, vias 0 -> 2
- net MISO: track 132.5 -> 134.3 mm, vias 3 -> 7
- net !SD_CD: track 92.5 -> 94.3 mm, vias 7 -> 11
- net USB_TXD: track 100.0 -> 99.3 mm
- net GND: vias 37 -> 48
Other:
- board text added: "+"
