File: LaserCutter.sch (EAGLE design)
At the start: 126 parts, among them IC1 ATMEGA8U2, IC10 LM393D, IC11 74AHC1G02DBV, IC12 74AHC1G02DBV, IC13 74AHC1G08DBV, IC14 MAX6675, IC2 BEE module, IC3 MC34063, IC4 74AHC1G02DBV, IC5 74AHC1G08DBV, IC6 ATMEGA2560-16AU, IC7 CD4050D, IC8 LD1117S33, IC9 OPA340N, J1 X Stepper, J10 Laser HV PSU, J11 24V in, J12 Interface, J13 I2C, J14 ISP, J15 SDMMC18650, J16 UART3, J17 X Home, J18 Z Home, J19 Y Home, J2 Reset En, J20 Interlocks, J21 Spare, J22 Omega PCC-SMP-V-K, J4 USB, J5 Y Stepper, J6 Ground, J7 ISP, J8 Z Stepper, J9 Stepper disable, Q1 16 MHz, Q2 16MHz

Commit message: foo
Parts:
- removed J22: Omega PCC-SMP-V-K, Thermocouple:TC_JACK
- added J3: USB, freetronics-master-v1:USB-FT
- J10: value Laser HV PSU -> 24V in; device con-phoenix-254:MPT4 -> con-wago-508:W237-02P
- J11: value 24V in -> Interface; device con-wago-508:W237-02P -> con-phoenix-254:MPT8
- J12: value Interface -> I2C; device con-phoenix-254:MPT8 -> freetronics-master-v1:M02PTH
- J13: value I2C -> SDMMC18650; device pinhead:PINHD-1X2 -> adafruit:SDMMC18650
- J14: device SparkFun:AVR_SPI_PRG_6NS -> freetronics-master-v1:PINHD-2X3
- J15: value SDMMC18650 -> UART3; device adafruit:SDMMC18650 -> freetronics-master-v1:M02PTH
- J16: value UART3 -> X Home; device pinhead:PINHD-1X2 -> con-phoenix-254:MPT3
- J17: value X Home -> Z Home; device con-phoenix-254:MPT3 -> con-phoenix-254:MPT5
- J18: value Z Home -> Y Home; device con-phoenix-254:MPT5 -> con-phoenix-254:MPT3
- J19: value Y Home -> Interlocks; device con-phoenix-254:MPT3 -> con-phoenix-254:MPT2
- J20: value Interlocks -> Spare
- J21: value Spare -> Omega PCC-SMP-V-K; device con-phoenix-254:MPT2 -> freetronics-luke:PCC-SMP-V
- J4: value USB -> Y Stepper; device freetronics-master-v1:USB-FT -> con-phoenix-254:MPT6
- J5: value Y Stepper -> Ground; device con-phoenix-254:MPT6 -> jumper:SJ
- J6: value Ground -> ISP; device jumper:SJ -> freetronics-master-v1:PINHD-2X3
- J7: value ISP -> Z Stepper; device SparkFun:AVR_SPI_PRG_6NS -> con-phoenix-254:MPT6
- J8: value Z Stepper -> Stepper disable; device con-phoenix-254:MPT6 -> wirepad:1,6/0,8
- J9: value Stepper disable -> Laser HV PSU; device wirepad:1,6/0,8 -> con-phoenix-254:MPT4
- renumbered $0000002 to $1
Connections:
- net !8U2_RESET: now also J6.5; no longer J7.5
- net !DOOR: now also J19-1.1, J9-2.1; no longer J10-2.1, J20-1.1
- net !LASER_ENABLE: now also J9-1.1; no longer J10-1.1
- net !SD_CD: now also J13.CARD_DETECT; no longer J15.CARD_DETECT
- net !UI_CS: now also J11-8.1; no longer J12-8.1
- net +24V: now also J10-1.KL, J16-1.1, J4-6.1, J7-6.1; no longer J11-1.KL, J19-1.1, J5-6.1, J8-6.1
- net +3V3: now also J13.VDD; no longer J15.VDD
- net +5V: now also J11-1.1, J17-2.1, J4-3.1, J6.2, J7-3.1; no longer J12-1.1, J18-2.1, J5-3.1, J7.2, J8-3.1
- net 8U2_MISO: now also J6.1; no longer J7.1
- net 8U2_MOSI: now also J6.4; no longer J7.4
- net 8U2_SCK: now also J6.3; no longer J7.3
- net GND: now also J10-2.KL, J11-2.1, J13.COMMON_SW, J13.GND, J13.VSS1, J13.VSS2, J16-3.1, J17-5.1, J18-3.1, J20-2.1, J21.GND, J21.T-, J4-5.1, J5.2, J6.6, J7-5.1, J9-3.1; no longer J10-3.1, J11-2.KL, J12-2.1, J15.COMMON_SW, J15.GND, J15.VSS1, J15.VSS2, J17-3.1, J18-5.1, J19-3.1, J21-2.1, J22.GND, J22.GND1, J22.T-, J5-5.1, J6.2, J7.6, J8-5.1
- net J81: now also J4-4.1, J7-4.1, J8.P; no longer J5-4.1, J8-4.1, J9.P
- net LASER_MODULATION: now also J9-4.1; no longer J10-4.1
- net MISO: now also J11-5.1, J13.DATA_OUT; no longer J12-5.1, J15.DATA_OUT
- net MOSI: now also J11-6.1; no longer J12-6.1
- net N$1: now also J13.DATA_IN; no longer J15.DATA_IN
- net N$101: now also J3.D-; no longer J4.D-
- net N$12: now also J19-2.1, J20-1.1; no longer J20-2.1, J21-1.1
- net N$120: now also J3.SH$1, J3.SH$2, J3.SH$3, J3.SH$4; no longer J4.SH$1, J4.SH$2, J4.SH$3, J4.SH$4
- net N$19: now also J13.CS; no longer J15.CS
- net N$25: now also J21.T+; no longer J22.T+
- net N$35: now also J17-3.1; no longer J18-3.1
- net N$6: now also J3.GND, J5.1; no longer J4.GND, J6.1
- net N$9: now also J13.SCLK; no longer J15.SCLK
- net N$97: now also J3.VBUS; no longer J4.VBUS
- net N$98: now also J3.D+; no longer J4.D+
- net RXD3: now also J15.1; no longer J16.1
- net SCK: now also J11-7.1; no longer J12-7.1
- net SCL: now also J12.2; no longer J13.2
- net SDA: now also J12.1; no longer J13.1
- net TXD3: now also J15.2; no longer J16.2
- net UI_RXD: now also J11-3.1; no longer J12-3.1
- net UI_TXD: now also J11-4.1; no longer J12-4.1
- net X_HOME: now also J16-2.1; no longer J17-2.1
- net Y_DIR: now also J4-2.1; no longer J5-2.1
- net Y_HOME: now also J18-2.1; no longer J19-2.1
- net Y_STEP: now also J4-1.1; no longer J5-1.1
- net Z_DIR: now also J7-2.1; no longer J8-2.1
- net Z_HOME: now also J17-4.1; no longer J18-4.1
- net Z_STEP: now also J7-1.1; no longer J8-1.1
Other:
- moved on the sheet: J20-1, J20-2

Commit message: a few tweaks
Connections:
- new net DAT1: J13.DAT1
- new net DAT2: J13.DAT2
- new net WP: J13.WRITE_PROTECT
Changed lines of the file:
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@@
 <setting verticaltext="up"/>
 </settings>
-<grid distance="0.1" unitdist="inch" unit="inch" style="lines" multiple="1" display="yes" altdistance="0.01" altunitdist="inch" altunit="inch"/>
+<grid distance="0.1" unitdist="inch" unit="inch" style="lines" multiple="1" display="no" altdistance="0.01" altunitdist="inch" altunit="inch"/>
 <layers>
-<layer number="1" name="Top" color="4" fill="1" visible="yes" active="no"/>
-<layer number="2" name="Route2" color="1" fill="3" visible="yes" active="no"/>
-<layer number="3" name="Route3" color="4" fill="3" visible="yes" active="no"/>
-<layer number="4" name="Route4" color="1" fill="4" visible="yes" active="no"/>
-<layer number="5" name="Route5" color="4" fill="4" visible="yes" active="no"/>
-<layer number="6" name="Route6" color="1" fill="8" visible="yes" active="no"/>
-<layer number="7" name="Route7" color="4" fill="8" visible="yes" active="no"/>
-<layer number="8" name="Route8" color="1" fill="2" visible="yes" active="no"/>
-<layer number="9" name="Route9" color="4" fill="2" visible="yes" active="no"/>
-<layer number="10" name="Route10" color="1" fill="7" visible="yes" active="no"/>
-<layer number="11" name="Route11" color="4" fill="7" visible="yes" active="no"/>
-<layer number="12" name="Route12" color="1" fill="5" visible="yes" active="no"/>
-<layer number="13" name="Route13" color="4" fill="5" visible="yes" active="no"/>
-<layer number="14" name="Route14" color="1" fill="6" visible="yes" active="no"/>
-<layer number="15" name="Route15" color="4" fill="6" visible="yes" active="no"/>
-<layer number="16" name="Bottom" color="1" fill="1" visible="yes" active="no"/>
-<layer number="17" name="Pads" color="2" fill="1" visible="yes" active="no"/>
-<layer number="18" name="Vias" color="2" fill="1" visible="yes" active="no"/>
-<layer number="19" name="Unrouted" color="6" fill="1" visible="yes" active="no"/>
-<layer number="20" name="Dimension" color="15" fill="1" visible="yes" active="no"/>
-<layer number="21" name="tPlace" color="7" fill="1" visible="yes" active="no"/>
-<layer number="22" name="bPlace" color="7" fill="1" visible="yes" active="no"/>
-<layer number="23" name="tOrigins" color="15" fill="1" visible="yes" active="no"/>
-<layer number="24" name="bOrigins" color="15" fill="1" visible="yes" active="no"/>
-<layer number="25" name="tNames" color="7" fill="1" visible="yes" active="no"/>
-<layer number="26" name="bNames" color="7" fill="1" visible="yes" active="no"/>
-<layer number="27" name="tValues" color="7" fill="1" visible="yes" active="no"/>
-<layer number="28" name="bValues" color="7" fill="1" visible="yes" active="no"/>
+<layer number="1" name="Top" color="4" fill="1" visible="no" active="no"/>
+<layer number="2" name="Route2" color="1" fill="3" visible="no" active="no"/>
+<layer number="3" name="Route3" color="4" fill="3" visible="no" active="no"/>
+<layer number="4" name="Route4" color="1" fill="4" visible="no" active="no"/>
+<layer number="5" name="Route5" color="4" fill="4" visible="no" active="no"/>
+<layer number="6" name="Route6" color="1" fill="8" visible="no" active="no"/>
+<layer number="7" name="Route7" color="4" fill="8" visible="no" active="no"/>
+<layer number="8" name="Route8" color="1" fill="2" visible="no" active="no"/>
+<layer number="9" name="Route9" color="4" fill="2" visible="no" active="no"/>
+<layer number="10" name="Route10" color="1" fill="7" visible="no" active="no"/>
+<layer number="11" name="Route11" color="4" fill="7" visible="no" active="no"/>
+<layer number="12" name="Route12" color="1" fill="5" visible="no" active="no"/>
+<layer number="13" name="Route13" color="4" fill="5" visible="no" active="no"/>
+<layer number="14" name="Route14" color="1" fill="6" visible="no" active="no"/>
+<layer number="15" name="Route15" color="4" fill="6" visible="no" active="no"/>
+<layer number="16" name="Bottom" color="1" fill="1" visible="no" active="no"/>
+<layer number="17" name="Pads" color="2" fill="1" visible="no" active="no"/>
+<layer number="18" name="Vias" color="2" fill="1" visible="no" active="no"/>
+<layer number="19" name="Unrouted" color="6" fill="1" visible="no" active="no"/>
+<layer number="20" name="Dimension" color="15" fill="1" visible="no" active="no"/>
+<layer number="21" name="tPlace" color="7" fill="1" visible="no" active="no"/>
+<layer number="22" name="bPlace" color="7" fill="1" visible="no" active="no"/>
+<layer number="23" name="tOrigins" color="15" fill="1" visible="no" active="no"/>
+<layer number="24" name="bOrigins" color="15" fill="1" visible="no" active="no"/>
+<layer number="25" name="tNames" color="7" fill="1" visible="no" active="no"/>
+<layer number="26" name="bNames" color="7" fill="1" visible="no" active="no"/>
+<layer number="27" name="tValues" color="7" fill="1" visible="no" active="no"/>
+<layer number="28" name="bValues" color="7" fill="1" visible="no" active="no"/>
 <layer number="29" name="tStop" color="7" fill="3" visible="no" active="no"/>
 <layer number="30" name="bStop" color="7" fill="6" visible="no" active="no"/>
@@
 <layer number="35" name="tGlue" color="7" fill="4" visible="no" active="no"/>
 <layer number="36" name="bGlue" color="7" fill="5" visible="no" active="no"/>
-<layer number="37" name="tTest" color="7" fill="1" visible="yes" active="no"/>
-<layer number="38" name="bTest" color="7" fill="1" visible="yes" active="no"/>
+<layer number="37" name="tTest" color="7" fill="1" visible="no" active="no"/>
+<layer number="38" name="bTest" color="7" fill="1" visible="no" active="no"/>
 <layer number="39" name="tKeepout" color="4" fill="11" visible="no" active="no"/>
 <layer number="40" name="bKeepout" color="1" fill="11" visible="no" active="no"/>
@@
 <layer number="44" name="Drills" color="7" fill="1" visible="no" active="no"/>
 <layer number="45" name="Holes" color="7" fill="1" visible="no" active="no"/>
-<layer number="46" name="Milling" color="3" fill="1" visible="yes" active="no"/>
-<layer number="47" name="Measures" color="7" fill="1" visible="yes" active="no"/>
-<layer number="48" name="Document" color="7" fill="1" visible="yes" active="no"/>
-<layer number="49" name="Reference" color="7" fill="1" visible="yes" active="no"/>
-<layer number="50" name="dxf" color="7" fill="1" visible="yes" active="no"/>
-<layer number="51" name="tDocu" color="7" fill="1" visible="yes" active="no"/>
-<layer number="52" name="bDocu" color="7" fill="1" visible="yes" active="no"/>
-<layer number="53" name="tGND_GNDA" color="7" fill="9" visible="yes" active="no"/>
-<layer number="54" name="bGND_GNDA" color="1" fill="9" visible="yes" active="no"/>
-<layer number="56" name="wert" color="7" fill="1" visible="yes" active="no"/>
-<layer number="60" name="p_dimension" color="6" fill="0" visible="yes" active="no"/>
-<layer number="61" name="pt_docu" color="7" fill="0" visible="yes" active="no"/>
+<layer number="46" name="Milling" color="3" fill="1" visible="no" active="no"/>
+<layer number="47" name="Measures" color="7" fill="1" visible="no" active="no"/>
+<layer number="48" name="Document" color="7" fill="1" visible="no" active="no"/>
+<layer number="49" name="Reference" color="7" fill="1" visible="no" active="no"/>
+<layer number="50" name="dxf" color="7" fill="1" visible="no" active="no"/>
+<layer number="51" name="tDocu" color="7" fill="1" visible="no" active="no"/>
+<layer number="52" name="bDocu" color="7" fill="1" visible="no" active="no"/>
+<layer number="53" name="tGND_GNDA" color="7" fill="9" visible="no" active="no"/>
+<layer number="54" name="bGND_GNDA" color="1" fill="9" visible="no" active="no"/>
+<layer number="56" name="wert" color="7" fill="1" visible="no" active="no"/>
+<layer number="60" name="p_dimension" color="6" fill="0" visible="no" active="no"/>
+<layer number="61" name="pt_docu" color="7" fill="0" visible="no" active="no"/>
 <layer number="91" name="Nets" color="2" fill="1" visible="yes" active="yes"/>
 <layer number="92" name="Busses" color="1" fill="1" visible="yes" active="yes"/>
@@
 </segment>
 </net>
+<net name="DAT1" class="0">
+<segment>
+<pinref part="J13" gate="G$1" pin="DAT1"/>
+<wire x1="43.18" y1="246.38" x2="44.196" y2="246.38" width="0.1524" layer="91"/>
+</segment>
+</net>
+<net name="DAT2" class="0">
+<segment>
+<pinref part="J13" gate="G$1" pin="DAT2"/>
+<wire x1="43.434" y1="243.84" x2="43.18" y2="243.84" width="0.1524" layer="91"/>
+<wire x1="43.18" y1="243.84" x2="44.196" y2="243.84" width="0.1524" layer="91"/>
+</segment>
+</net>
+<net name="WP" class="0">
+<segment>
+<pinref part="J13" gate="G$1" pin="WRITE_PROTECT"/>
+<wire x1="43.18" y1="261.62" x2="43.434" y2="261.62" width="0.1524" layer="91"/>
+</segment>
+</net>
